File: Schematics/GPS_Module/GPS_Module.kicad_pcb (KiCad board)
At the start: 4 copper layers, 69.5 x 60 mm, 70 parts, among them J1 GT8E-6P-2H(55), J2 SWD_01x04_Pin, J4 Stack Male Edge Connector, J6 USB_C_Female_USB2_Small, SW1 SW_STM_RESET, SW2 SW_STM_BOOT_MODE, U1 STM32F103CBT6, U10 AMS1117-3.3, U2 CP2102N-Axx-xQFN28, U3 W25Q128JVS, U4 LM66100DCKR, U5 LM66100DCKR, U6 LM66100DCKR, U7 TPM8837C-SO1R, U9 ISO1042BQDWVR, Y1 X322516MMB4SI

Commit message: prepare for dedicated av-recovery repo (GPS & Altimter only)
Parts:
- R7: value 680R -> 680
Connections:
- J4 pad A12: unconnected-(J4-GND_B-PadA12) -> unconnected-(J4-GND_B-PadA12)_2
- J4 pad A7: unconnected-(J4-3.3V_B-PadA7) -> unconnected-(J4-3.3V_B-PadA7)_1
- J4 pad A9: unconnected-(J4-GND_B-PadA12) -> unconnected-(J4-GND_B-PadA12)_4
- J4 pad B10: unconnected-(J4-GND_B-PadA12) -> unconnected-(J4-GND_B-PadA12)_3
- J4 pad B11: unconnected-(J4-GND_B-PadA12) -> unconnected-(J4-GND_B-PadA12)_1
- J4 pad B8: unconnected-(J4-BATT_B-PadB7) -> unconnected-(J4-BATT_B-PadB7)_2
- J4 pad B9: unconnected-(J4-BATT_B-PadB7) -> unconnected-(J4-BATT_B-PadB7)_1
